File: MASA-Radio Board.kicad_pcb (KiCad board)
At the start: 4 copper layers, 75.8 x 76.2 mm, 104 parts, among them IC1 FAN4010IL6X_F113, IC2 FAN4010IL6X_F113, J1 Conn_01x02, J2 Conn_01x02_Male, J3 Conn_01x02_Male, J4 Conn_01x03_Male, J5 Conn_01x06, J6 SC_19-20, J7 Conn_01x06, J8 Conn_01x02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

Commit message: Fixed drc
Parts:
- moved C5 3.12 mm to (162.1, 114.1)
Routing:
- net USB_VBUS: track 35.3 -> 30.8 mm
- net GND: track 101.9 -> 98.1 mm
Changed lines of the file:
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@@
-(kicad_pcb (version 20171130) (host pcbnew "(5.1.4)-1")
+(kicad_pcb (version 20171130) (host pcbnew "(5.1.5)-3")
   (general
     (thickness 1.6)
     (drawings 18)
-    (tracks 956)
+    (tracks 951)
     (zones 0)
     (modules 104)
@@
   )
   (module Capacitor_SMD:C_0603_1608Metric (layer F.Cu)
-    (at 162.179 117.221 270)
+    (at 162.1 114.1 270)
     (descr "Capacitor SMD 0603 (1608 Metric), square (rectangular) end terminal, IPC_7351 nominal, (Body size source: http://www.tortai-tech.com/upload/download/2011102023233369053.pdf), generated with kicad-footprint-generator")
     (tags capacitor)
@@
   (via (at 158.623 118.364) (size 0.8) (drill 0.4) (layers F.Cu B.Cu) (net 1))
   (segment (start 157.31 118.364) (end 158.623 118.364) (width 0.381) (layer F.Cu) (net 1))
-  (segment (start 162.179 118.0085) (end 162.179 118.237) (width 0.381) (layer F.Cu) (net 1))
   (via (at 163.703 118.364) (size 0.8) (drill 0.4) (layers F.Cu B.Cu) (net 1))
-  (segment (start 162.179 118.237) (end 163.576 118.237) (width 0.381) (layer F.Cu) (net 1))
   (segment (start 171.935 125.857) (end 172.085 126.007) (width 0.2032) (layer F.Cu) (net 1))
   (segment (start 170.919 125.857) (end 171.935 125.857) (width 0.2032) (layer F.Cu) (net 1))
@@
   (via (at 171.45 119.38) (size 0.8) (drill 0.4) (layers F.Cu B.Cu) (net 1))
   (segment (start 171.45 120.331) (end 171.45 119.38) (width 0.254) (layer F.Cu) (net 1))
-  (segment (start 160.604 116.4335) (end 162.179 118.0085) (width 0.254) (layer F.Cu) (net 1))
   (segment (start 160.528 116.4335) (end 160.604 116.4335) (width 0.254) (layer F.Cu) (net 1))
   (segment (start 153.3145 117.729) (end 153.3145 116.6875) (width 0.254) (layer F.Cu) (net 1))
@@
   (segment (start 150.368 112.068) (end 150.3 112) (width 0.381) (layer F.Cu) (net 20))
   (segment (start 150.368 113.284) (end 150.368 112.068) (width 0.381) (layer F.Cu) (net 20))
-  (segment (start 150.368 113.849685) (end 152.232717 115.714402) (width 0.2032) (layer In2.Cu) (net 20))
-  (segment (start 150.368 113.284) (end 150.368 113.849685) (width 0.2032) (layer In2.Cu) (net 20))
-  (segment (start 152.232717 115.714402) (end 158.732598 115.714402) (width 0.2032) (layer In2.Cu) (net 20))
-  (segment (start 171.812681 102.634319) (end 178.013247 102.634319) (width 0.2032) (layer In2.Cu) (net 20))
-  (segment (start 158.732598 115.714402) (end 171.812681 102.634319) (width 0.2032) (layer In2.Cu) (net 20))
+  (segment (start 150.368 113.849685) (end 150.368 113.284) (width 0.2032) (layer In2.Cu) (net 20))
+  (segment (start 152.272416 115.754101) (end 150.368 113.849685) (width 0.2032) (layer In2.Cu) (net 20))
+  (segment (start 158.692899 115.754101) (end 152.272416 115.754101) (width 0.2032) (layer In2.Cu) (net 20))
+  (segment (start 171.812681 102.634319) (end 158.692899 115.754101) (width 0.2032) (layer In2.Cu) (net 20))
+  (segment (start 178.013247 102.634319) (end 171.812681 102.634319) (width 0.2032) (layer In2.Cu) (net 20))
   (segment (start 123.825 107.823) (end 123.825 116.508) (width 0.2032) (layer F.Cu) (net 21))
   (segment (start 126.048 105.6) (end 123.825 107.823) (width 0.2032) (layer F.Cu) (net 21))
@@
   (segment (start 142.4155 120.1165) (end 141.859 119.56) (width 0.2032) (layer F.Cu) (net 35))
   (segment (start 144.145 120.1165) (end 142.4155 120.1165) (width 0.2032) (layer F.Cu) (net 35))
-  (segment (start 162.179 115.996) (end 161.372 115.189) (width 0.25) (layer F.Cu) (net 45))
-  (segment (start 162.179 116.4335) (end 162.179 115.996) (width 0.25) (layer F.Cu) (net 45))
   (segment (start 156.7 112.5) (end 156.7 112) (width 0.25) (layer F.Cu) (net 45))
-  (segment (start 159.389 115.189) (end 156.7 112.5) (width 0.25) (layer F.Cu) (net 45))
-  (segment (start 161.372 115.189) (end 159.389 115.189) (width 0.25) (layer F.Cu) (net 45))
-  (segment (start 162.179 113.271) (end 162.179 116.4335) (width 0.2032) (layer F.Cu) (net 45))
   (segment (start 169.95 105.5) (end 162.179 113.271) (width 0.2032) (layer F.Cu) (net 45))
   (segment (start 171.280616 105.5) (end 171.2 105.5) (width 0.2032) (layer F.Cu) (net 45))
@@
   (segment (start 179.66 112.53) (end 179.66 111.53) (width 0.2032) (layer F.Cu) (net 45))
   (segment (start 171.2 105.5) (end 173.27 105.5) (width 0.2032) (layer F.Cu) (net 45))
+  (segment (start 156.7 112.5) (end 156.7 112.8) (width 0.2032) (layer F.Cu) (net 45))
+  (segment (start 157.171 113.271) (end 162.179 113.271) (width 0.2032) (layer F.Cu) (net 45))
+  (segment (start 156.7 112.8) (end 157.171 113.271) (width 0.2032) (layer F.Cu) (net 45))
   (segment (start 161.1258 99.5045) (end 160.02 100.6103) (width 0.2032) (layer F.Cu) (net 56))
   (segment (start 162.179 99.5045) (end 161.1258 99.5045) (width 0.2032) (layer F.Cu) (net 56))
